File: tmc5130-uart/interface.kicad_sch (KiCad schematic)
At the start: 12 parts, among them J301 FFC_P1mm_BOT_RA_SMD, M301 Fan_5VDC_25x25x8mm, U301 TPSM365R6V5RDNR

Commit message: Add components
Parts:
- removed C305: 1uF_25V, Janelia:C_0402_1005Metric, symbol Janelia:C_1uF_25V_0402
- removed D302: D_Zener_47V_1W, Janelia:D_SMA, symbol Janelia:D_Zener_47V_1W
- removed D304: D, Janelia:D_SMB, symbol Janelia:D_1.25V@2A_400V
- removed M301: Fan_5VDC_25x25x8mm, Janelia:FAN_5VDC_25x25x8mm, symbol Janelia:Fan_5VDC_25x25x8mm
- removed R302: 0.24, Janelia:R_2512_6332Metric, symbol Janelia:R_0.240_1W_2512
- added R302: 120, Janelia:R_0402_1005Metric, symbol Janelia:R_120_0402
- renumbered C304 to C302, C302 to C303, C303 to C304
Connections:
- net SWN: now also R302.2
- net SWP: now also R302.1
- net VAA: now also C301.1, C302.1, U301.2 (EN), U301.3 (VIN)
- net VCC: now also U301.11 (MODE_SYNC), U301.8 (VCC); no longer C301.1, C302.1, U301.2 (EN), U301.3 (VIN)
- net VDD: no longer U301.11 (MODE_SYNC), U301.8 (VCC)
