File: prism-pcb/interface.kicad_sch (KiCad schematic)
At the start: 21 parts, among them J301 USB_C_Receptacle_USB2.0_16P_G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, M301 Fan_5VDC_25x25x8mm, U301 TPSM365R6V5RDNR, U302 LTC6820HMS-TRPBF

Commit message: Preliminary routing for v2.0
Parts:
- removed M301: Fan_5VDC_25x25x8mm, Janelia:FAN_5VDC_25x25x8mm, symbol Janelia:Fan_5VDC_25x25x8mm
- removed R301: 120, Janelia:R_0402_1005Metric, symbol Janelia:R_120_0402
- added R301: 100, Janelia:R_0402_1005Metric, symbol Janelia:R_100_0402
Connections:
- net IM renamed I0-
- net IM1 renamed I1-
- net IM2 renamed I2-
- net I2-: now also R301.2
- net IP renamed I0+
- net IP1 renamed I1+
- net IP2 renamed I2+
- net I2+: now also R301.1
Other:
- note added: "USB C Cable Differential Impedance 90 Ohm"
Changed lines of the file:
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@@
   (title_block
     (title "prism-pcb")
-    (date "2024-09-23")
+    (date "2024-09-26")
     (rev "2.0")
     (company "Howard Hughes Medical Institute")
@@
     (stroke (width 0) (type default))
   )
-  (wire (pts (xy 238.76 120.65) (xy 238.76 123.19))
-    (stroke (width 0) (type default))
-  )
   (wire (pts (xy 59.69 60.96) (xy 57.15 60.96))
     (stroke (width 0) (type default))
@@
   )
   (wire (pts (xy 157.48 147.32) (xy 154.94 147.32))
-    (stroke (width 0) (type default))
-  )
-  (wire (pts (xy 238.76 102.87) (xy 238.76 100.33))
     (stroke (width 0) (type default))
   )
@@
     (effects (font (size 1.27 1.27)) (justify right bottom))
   )
-  (label "IP1" (at 194.31 139.7 180) (fields_autoplaced)
+  (text "USB C Cable\nDifferential Impedance\n90 Ohm" (at 147.32 158.75 90)
+    (effects (font (size 1.27 1.27)) (justify right bottom))
+  )
+  (label "I1+" (at 194.31 139.7 180) (fields_autoplaced)
     (effects (font (size 1.27 1.27)) (justify right bottom))
   )
@@
     (effects (font (size 1.27 1.27)) (justify right bottom))
   )
-  (label "IP" (at 214.63 139.7 0) (fields_autoplaced)
-    (effects (font (size 1.27 1.27)) (justify left bottom))
-  )
-  (label "IP2" (at 144.78 135.89 90) (fields_autoplaced)
+  (label "I0+" (at 214.63 139.7 0) (fields_autoplaced)
+    (effects (font (size 1.27 1.27)) (justify left bottom))
+  )
+  (label "I2+" (at 144.78 135.89 90) (fields_autoplaced)
     (effects (font (size 1.27 1.27)) (justify left bottom))
   )
@@
     (effects (font (size 1.27 1.27)) (justify right bottom))
   )
-  (label "IM" (at 214.63 149.86 0) (fields_autoplaced)
+  (label "I0-" (at 214.63 149.86 0) (fields_autoplaced)
     (effects (font (size 1.27 1.27)) (justify left bottom))
   )
@@
     (effects (font (size 1.27 1.27)) (justify right bottom))
   )
-  (label "GND" (at 238.76 123.19 270) (fields_autoplaced)
-    (effects (font (size 1.27 1.27)) (justify right bottom))
-  )
   (label "VAA" (at 115.57 59.69 90) (fields_autoplaced)
     (effects (font (size 1.27 1.27)) (justify left bottom))
@@
     (effects (font (size 1.27 1.27)) (justify left bottom))
   )
-  (label "IM1" (at 194.31 149.86 180) (fields_autoplaced)
+  (label "I1-" (at 194.31 149.86 180) (fields_autoplaced)
     (effects (font (size 1.27 1.27)) (justify right bottom))
   )
@@
     (effects (font (size 1.27 1.27)) (justify right bottom))
   )
-  (label "IP" (at 50.8 101.6 0) (fields_autoplaced)
+  (label "I0+" (at 50.8 101.6 0) (fields_autoplaced)
     (effects (font (size 1.27 1.27)) (justify left bottom))
   )
@@
     (effects (font (size 1.27 1.27)) (justify right bottom))
   )
-  (label "IM2" (at 154.94 147.32 180) (fields_autoplaced)
-    (effects (font (size 1.27 1.27)) (justify right bottom))
-  )
-  (label "IM1" (at 170.18 147.32 0) (fields_autoplaced)
-    (effects (font (size 1.27 1.27)) (justify left bottom))
-  )
-  (label "IM" (at 50.8 93.98 0) (fields_autoplaced)
+  (label "I2-" (at 154.94 147.32 180) (fields_autoplaced)
+    (effects (font (size 1.27 1.27)) (justify right bottom))
+  )
+  (label "I1-" (at 170.18 147.32 0) (fields_autoplaced)
+    (effects (font (size 1.27 1.27)) (justify left bottom))
+  )
+  (label "I0-" (at 50.8 93.98 0) (fields_autoplaced)
     (effects (font (size 1.27 1.27)) (justify left bottom))
   )
@@
     (effects (font (size 1.27 1.27)) (justify left bottom))
   )
-  (label "IP2" (at 135.89 140.97 0) (fields_autoplaced)
+  (label "I2+" (at 135.89 140.97 0) (fields_autoplaced)
     (effects (font (size 1.27 1.27)) (justify left bottom))
   )
@@
     (effects (font (size 1.27 1.27)) (justify right bottom))
   )
-  (label "IP1" (at 170.18 142.24 0) (fields_autoplaced)
+  (label "I1+" (at 170.18 142.24 0) (fields_autoplaced)
     (effects (font (size 1.27 1.27)) (justify left bottom))
   )
@@
     (effects (font (size 1.27 1.27)) (justify right bottom))
   )
-  (label "+5V" (at 238.76 100.33 90) (fields_autoplaced)
-    (effects (font (size 1.27 1.27)) (justify left bottom))
-  )
-  (label "IM2" (at 135.89 148.59 0) (fields_autoplaced)
+  (label "I2-" (at 135.89 148.59 0) (fields_autoplaced)
     (effects (font (size 1.27 1.27)) (justify left bottom))
   )
@@
     (effects (font (size 1.27 1.27)) (justify right bottom))
   )
-  (label "IP" (at 50.8 99.06 0) (fields_autoplaced)
+  (label "I0+" (at 50.8 99.06 0) (fields_autoplaced)
     (effects (font (size 1.27 1.27)) (justify left bottom))
   )
@@
     (effects (font (size 1.27 1.27)) (justify right bottom))
   )
-  (label "IM2" (at 144.78 153.67 270) (fields_autoplaced)
+  (label "I2-" (at 144.78 153.67 270) (fields_autoplaced)
     (effects (font (size 1.27 1.27)) (justify right bottom))
   )
@@
     (effects (font (size 1.27 1.27)) (justify right bottom))
   )
-  (label "IP2" (at 154.94 142.24 180) (fields_autoplaced)
+  (label "I2+" (at 154.94 142.24 180) (fields_autoplaced)
     (effects (font (size 1.27 1.27)) (justify right bottom))
   )
@@
     (effects (font (size 1.27 1.27)) (justify right bottom))
   )
-  (label "IM" (at 50.8 96.52 0) (fields_autoplaced)
+  (label "I0-" (at 50.8 96.52 0) (fields_autoplaced)
     (effects (font (size 1.27 1.27)) (justify left bottom))
   )
@@
     )
   )
-  (symbol (lib_id "Janelia:R_120_0402") (at 144.78 144.78 0) (unit 1)
-    (in_bom yes) (on_board yes) (dnp no)
+  (symbol (lib_id "Janelia:R_100_0402") (at 144.78 144.78 0) (unit 1)
+    (in_bom yes) (on_board yes) (dnp no) (fields_autoplaced)
     (property "Reference" "R301" (at 146.05 144.78 0) (do_not_autoplace)
       (effects (font (size 1.016 1.016)) (justify left))
     )
-    (property "Value" "120" (at 144.78 144.78 90) (do_not_autoplace)
+    (property "Value" "100" (at 144.78 144.78 90) (do_not_autoplace)
       (effects (font (size 0.762 0.762)))
     )
@@
       (effects (font (size 1.524 1.524)) hide)
     )
-    (property "Vendor Part Number" "C114758" (at 151.892 139.7 90)
-      (effects (font (size 1.524 1.524)) hide)
-    )
-    (property "Synopsis" "RES SMD 120 OHM 1% 62.5mW" (at 154.432 137.16 90)
+    (property "Vendor Part Number" "C25076" (at 151.892 139.7 90)
+      (effects (font (size 1.524 1.524)) hide)
+    )
+    (property "Synopsis" "RES SMD 100 OHM 1% 62.5mW" (at 154.432 137.16 90)
       (effects (font (size 1.524 1.524)) hide)
     )
@@
       (effects (font (size 1.27 1.27)) hide)
     )
-    (property "Manufacturer" "YAGEO" (at 144.78 144.78 0)
-      (effects (font (size 1.27 1.27)) hide)
-    )
-    (property "Manufacturer Part Number" "RC0402FR-07120RL" (at 144.78 144.78 0)
-      (effects (font (size 1.27 1.27)) hide)
-    )
-    (property "LCSC" "C114758" (at 144.78 144.78 0)
+    (property "Manufacturer" "UNI-ROYAL(Uniroyal Elec)" (at 144.78 144.78 0)
+      (effects (font (size 1.27 1.27)) hide)
+    )
+    (property "Manufacturer Part Number" "0402WGF1000TCE" (at 144.78 144.78 0)
+      (effects (font (size 1.27 1.27)) hide)
+    )
+    (property "LCSC" "C25076" (at 144.78 144.78 0)
       (effects (font (size 1.27 1.27)) hide)
     )
@@
         )
       )
-    )
-  )
-  (symbol (lib_id "Janelia:Fan_5VDC_25x25x8mm") (at 238.76 111.76 0) (unit 1)
-    (in_bom no) (on_board yes) (dnp no) (fields_autoplaced)
-    (property "Reference" "M301" (at 242.57 111.76 0) (do_not_autoplace)
-      (effects (font (size 1.27 1.27)) (justify left))
-    )
-    (property "Value" "Fan_5VDC_25x25x8mm" (at 238.76 106.68 0) (do_not_autoplace)
-      (effects (font (size 1.27 1.27)) (justify top) hide)
-    )
-    (property "Footprint" "Janelia:FAN_5VDC_25x25x8mm" (at 238.76 93.98 0)
-      (effects (font (size 1.27 1.27)) hide)
-    )
-    (property "Datasheet" "~" (at 238.76 95.25 0)
-      (effects (font (size 1.27 1.27)) hide)
-    )
-    (property "Synopsis" "FAN AXIAL 25X8MM 5VDC WIRE" (at 238.76 105.41 0)
-      (effects (font (size 1.27 1.27)) hide)
-    )
-    (property "Manufacturer" "ebm-papst Inc." (at 238.76 102.87 0)
-      (effects (font (size 1.27 1.27)) hide)
-    )
-    (property "Manufacturer Part Number" "255M" (at 238.76 104.14 0) (do_not_autoplace)
-      (effects (font (size 1.27 1.27)) hide)
-    )
-    (property "Vendor" "Digi-Key" (at 238.76 100.33 0)
-      (effects (font (size 1.27 1.27)) hide)
-    )
-    (property "Vendor Part Number" "381-2353-ND" (at 238.76 97.79 0)
-      (effects (font (size 1.27 1.27)) hide)
-    )
-    (property "LCSC" "" (at 238.76 111.76 0)
-      (effects (font (size 1.27 1.27)) hide)
-    )
-    (property "Sim.Enable" "0" (at 238.76 111.76 0)
-      (effects (font (size 1.27 1.27)) hide)
-    )
-    (pin "3")
-    (pin "1")
-    (pin "2")
-    (instances
-      (project "prism-pcb"
-        (path "/df2b2e89-e055-4140-95de-f1df723db034/c1dd8f61-494c-402f-8e59-08309c64fc3f"
-          (reference "M301") (unit 1)
-        )
-      )
