File: prism-pcb/prism-pcb.kicad_pcb (KiCad board)
At the start: 2 copper layers, 40 x 40 mm, 47 parts, among them J301 USB_C_Receptacle_USB2.0_16P_G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, J401 Molex_Pico-SPOX_Horizontal, M301 Fan_5VDC_25x25x8mm, U301 TPSM365R6V5RDNR, U302 LTC6820HMS-TRPBF, U401 TMC5130A-TA, X401 16MHz

Commit message: Preliminary routing for v2.0
Parts:
- removed M301: Fan_5VDC_25x25x8mm, Janelia:FAN_5VDC_25x25x8mm
- C306, C307, C308, FL301, R303, R304, R305, TR301, U302: moved to F.Cu
- R301: value 120 -> 100; moved to F.Cu
- moved C303 31.6 mm to (169.4, 91.1), turned to 180 degrees
- moved C301 29.8 mm to (162.9, 91.3), turned to 90 degrees
- moved U301 26.2 mm to (167.9, 94.6), turned to 0 degrees
- moved C302 22.1 mm to (165.2, 93.3), turned to 90 degrees
- moved C305 21.1 mm to (163.7, 96.1), turned to -90 degrees
- moved C304 20.2 mm to (165.2, 95.6), turned to -90 degrees
- moved C308 17.6 mm to (137.7, 107.6)
- moved TR301 17.4 mm to (136.9, 111.3), turned to 90 degrees
- moved D301 16.8 mm to (135.9, 94.8)
- moved R302 16.8 mm to (138.9, 94.8)
- moved FL301 16.3 mm to (141.7, 111.3), turned to -90 degrees
- moved C307 9.57 mm to (139.7, 107.6), turned to 180 degrees
- moved R305 7.72 mm to (146.2, 101.3), turned to 90 degrees
- moved C306 6.86 mm to (141.9, 100.3)
- moved R301 6.60 mm to (141.7, 107.6), turned to 180 degrees
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Connections:
- net /interface/IM renamed /interface/I0-
- net /interface/IM1 renamed /interface/I1-
- net /interface/IM2 renamed /interface/I2-
- net /interface/IP renamed /interface/I0+
- net /interface/IP1 renamed /interface/I1+
- net /interface/IP2 renamed /interface/I2+
Routing:
- net /VAA: track 54.7 -> 107.5 mm, vias 0 -> 2
- net /GND: track 295.1 -> 341.7 mm, vias 3 -> 5
- net /interface/I0-: track 0.00 -> 16.0 mm
- net /interface/I0+: track 0.00 -> 15.5 mm
- net /+5V: track 72.7 -> 65.6 mm, vias 0 -> 2
- net /interface/I1+: track 0.00 -> 6.33 mm
- net /COPI: track 9.97 -> 4.67 mm, vias 1 -> 0
- net /CIPO: track 10.0 -> 6.53 mm, vias 1 -> 0
- net /interface/I1-: track 0.00 -> 3.47 mm
- net /interface/CT: track 0.00 -> 2.78 mm
- net /~{CS}: track 8.85 -> 6.58 mm, vias 1 -> 0
- net /interface/ICMP: track 4.00 -> 2.41 mm
- net /interface/I2+: track 1.78 -> 3.21 mm
- net /interface/I2-: track 2.00 -> 3.43 mm
- net /SCK: track 6.61 -> 5.78 mm, vias 1 -> 0
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